File: BACKPACK/BACKPACK.kicad_sch (KiCad schematic)
At the start: 16 parts, among them J4 Conn_Coaxial, U10 RAK3172, U9 TESEO-LIV4F

Commit message: small fixes, started working on the backpack
Parts:
- added H1, H2, H3, H4, H5, H6: MountingHole, MountingHole:MountingHole_3.2mm_M3, symbol Mechanical:MountingHole
- added J5, J6: Conn_02x08_Odd_Even, Connector_PinHeader_2.54mm:PinHeader_2x08_P2.54mm_Vertical, symbol Connector_Generic:Conn_02x08_Odd_Even
- added R7: 1k, Resistor_SMD:R_0603_1608Metric_Pad0.98x0.95mm_HandSolder, symbol Device:R_Small
- added SW1: BOOTSEL, TSB008:TSB008, symbol Switch:SW_Push
- added SW2: RESET, TSB008:TSB008, symbol Switch:SW_Push
Connections:
- net +3V3: now also J5.1 (Pin_1), J5.2 (Pin_2), J6.1 (Pin_1), J6.2 (Pin_2)
- net GND: now also J5.13 (Pin_13), J5.14 (Pin_14), J5.7 (Pin_7), J6.15 (Pin_15), J6.16 (Pin_16), R7.1, SW1.1
- net PPS: now also J6.4 (Pin_4)
- net RX_GPS: now also J5.9 (Pin_9)
- net SCL_RADIO: now also J5.16 (Pin_16)
- net SDA_RADIO: now also J5.15 (Pin_15)
- net TX_GPS: now also J5.10 (Pin_10)
- new net: R7.2, SW2.1
- new net BOOTSEL: J6.6 (Pin_6), SW1.2
- new net CPU_SWDCLK: J6.3 (Pin_3)
- new net CPU_SWDIO: J6.5 (Pin_5)
- new net GPIO20: J5.8 (Pin_8)
- new net GPIO39: J6.7 (Pin_7)
- new net GPIO41: J6.9 (Pin_9)
- new net GPIO42: J6.10 (Pin_10)
- new net GPIO43: J6.11 (Pin_11)
- new net GPIO44: J6.12 (Pin_12)
- new net GPIO45: J6.14 (Pin_14)
- new net GPIO46: J6.13 (Pin_13)
- new net HIL_RX: J5.12 (Pin_12)
- new net HIL_TX: J5.11 (Pin_11)
- new net PWM1: J5.4 (Pin_4)
- new net PWM2: J5.5 (Pin_5)
- new net PWM3: J5.6 (Pin_6)
- new net PWM4: J5.3 (Pin_3)
- new net RESET: J6.8 (Pin_8), SW2.2

Commit message: aiuto
Parts:
- removed JP1: SolderJumper_2_Open, Jumper:SolderJumper-2_P1.3mm_Open_TrianglePad1.0x1.5mm, symbol Jumper:SolderJumper_2_Open
- added J1, J2, J3, J7: Conn_01x03_Pin, Connector_JST:JST_XH_B3B-XH-A_1x03_P2.50mm_Vertical, symbol Connector:Conn_01x03_Pin
Connections:
- net CPU_SWDCLK: now also J2.1 (Pin_1)
- net CPU_SWDIO: now also J2.2 (Pin_2)
- net GND: now also J1.3 (Pin_3), J2.3 (Pin_3), J3.3 (Pin_3), J7.3 (Pin_3)
- net HIL_RX: now also J1.2 (Pin_2)
- net HIL_TX: now also J1.1 (Pin_1)
- net SWCLK_RADIO: now also J3.2 (Pin_2)
- net SWDIO_RADIO: now also J3.1 (Pin_1)
- net UART1_RX_RADIO: now also J7.1 (Pin_1)
- net UART1_TX_RADIO: now also J7.2 (Pin_2)
- no-connect marks 17 -> 18
