File: BACKPACK/BACKPACK.kicad_pcb (KiCad board)
At the start: 2 copper layers, 70.8 x 45 mm, 23 parts, among them J4 Conn_Coaxial, J5 Conn_02x06_Counter_Clockwise, U10 RAK3172, U9 TESEO-LIV4F

Commit message: small fixes, started working on the backpack
Parts:
- removed ? (x4): , 
- removed the J5 at (176.9, 79.2)
- removed the J5 at (141.6, 79.2)
- removed the J5 at (164.1, 70.8)
- added H1: MountingHole, MountingHole:MountingHole_3.2mm_M3, F.Cu at (131.0, 70.0)
- added H2: MountingHole, MountingHole:MountingHole_3.2mm_M3, F.Cu at (192.8, 69.8)
- added H3: MountingHole, MountingHole:MountingHole_3.2mm_M3, F.Cu at (131.0, 106.0)
- added H4: MountingHole, MountingHole:MountingHole_3.2mm_M3, F.Cu at (192.5, 106.0)
- added H5: MountingHole, MountingHole:MountingHole_3.2mm_M3, F.Cu at (185.0, 106.0)
- added H6: MountingHole, MountingHole:MountingHole_3.2mm_M3, F.Cu at (138.5, 70.0)
- added J5: Conn_02x08_Odd_Even, Connector_PinHeader_2.54mm:PinHeader_2x08_P2.54mm_Vertical, B.Cu at (177.0, 76.8)
- added J6: Conn_02x08_Odd_Even, Connector_PinHeader_2.54mm:PinHeader_2x08_P2.54mm_Vertical, B.Cu at (141.7, 76.7)
- added R7: 1k, Resistor_SMD:R_0603_1608Metric_Pad0.98x0.95mm_HandSolder, F.Cu at (131.0, 75.8)
- added SW1: BOOTSEL, TSB008:TSB008, F.Cu at (133.0, 80.8)
- added SW2: RESET, TSB008:TSB008, F.Cu at (128.9, 80.8)
- C39, JP1: moved to B.Cu
- moved D11 22.5 mm to (137.8, 108.5), turned to 90 degrees
- moved RN1 22.1 mm to (139.1, 104.6), turned to -90 degrees
- moved JP1 17.0 mm to (168.5, 88.2)
- moved D10 16.6 mm to (140.8, 108.5), turned to 90 degrees
- moved D9 14.4 mm to (143.8, 108.5), turned to 90 degrees
- moved TP1 14.0 mm to (158.3, 76.6)
- moved U9 14.0 mm to (165.8, 81.0)
- moved U10 11.3 mm to (155.8, 101.3)
- moved C39 9.28 mm to (165.8, 106.2), turned to 90 degrees
- moved BT1 2.69 mm to (174.1, 100.3)
- moved C37 1.90 mm to (188.0, 98.0)
- moved C40 1.90 mm to (183.6, 96.8)
- moved D8 1.90 mm to (180.0, 98.0)
- moved R39 1.90 mm to (183.6, 99.3)
- moved J4 1.40 mm to (127.2, 97.8)
Routing:
- net /SDA_RADIO: track 0.00 -> 58.4 mm
- net /SCL_RADIO: track 0.00 -> 58.3 mm, vias 0 -> 2
- net /RX_GPS: track 0.00 -> 56.5 mm, vias 0 -> 1
- net /TX_GPS: track 0.00 -> 51.6 mm, vias 0 -> 1
- net Net-(BT1-+): track 0.00 -> 36.8 mm, vias 0 -> 1
- net PPS: track 0.00 -> 35.4 mm
- net /L_RED: track 0.00 -> 24.3 mm, vias 0 -> 1
- net /L_BLUE: track 0.00 -> 20.5 mm, vias 0 -> 1
- net /L_GREEN: track 0.00 -> 19.8 mm, vias 0 -> 1
- net ANT: track 0.00 -> 18.8 mm, vias 0 -> 1
- net /RESET: track 0.00 -> 12.7 mm
- net /BOOTSEL: track 0.00 -> 7.89 mm
- net Net-(JP1-A): track 0.00 -> 7.56 mm
- net Net-(D11-A): track 0.00 -> 4.88 mm
- net Net-(D9-A): track 0.00 -> 4.69 mm
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- added copper zone on In2.Cu, net +3V3
- added copper zone on In1.Cu, net GND
Other:
- copper layers 2 -> 4
- board text added: "16"
- board text added: "17"
- board text added: "20"
- board text added: "24"
- board text added: "25"
- board text added: "26"
- board text added: "27"
- board text added: "39"
- board text added: "3V3"
- board text added: "41"
- board text added: "42"
- board text added: "43"
- board text added: "44"
- board text added: "45"
- board text added: "46"
- board text added: "8"
- board text added: "9"
- board text added: "BOOT"
- board text added: "GND"
- board text added: "RESET"
- board text added: "SCL"
- board text added: "SDA"
- board text added: "SWDCK"
- board text added: "SWDIO"

Commit message: aiuto
Parts:
- removed JP1: SolderJumper_2_Open, Jumper:SolderJumper-2_P1.3mm_Open_TrianglePad1.0x1.5mm
- added J1: Conn_01x03_Pin, Connector_JST:JST_XH_B3B-XH-A_1x03_P2.50mm_Vertical, F.Cu at (184.7, 93.4)
- added J2: Conn_01x03_Pin, Connector_JST:JST_XH_B3B-XH-A_1x03_P2.50mm_Vertical, F.Cu at (191.9, 82.2)
- added J3: Conn_01x03_Pin, Connector_JST:JST_XH_B3B-XH-A_1x03_P2.50mm_Vertical, F.Cu at (184.7, 82.2)
- added J7: Conn_01x03_Pin, Connector_JST:JST_XH_B3B-XH-A_1x03_P2.50mm_Vertical, F.Cu at (191.9, 93.4)
- U10: moved to F.Cu
- moved D10 30.3 mm to (171.1, 108.7)
- moved D11 30.3 mm to (168.1, 108.7)
- moved D9 30.3 mm to (174.1, 108.7)
- moved RN1 30.3 mm to (169.4, 104.8)
- moved C39 10.0 mm to (165.1, 96.3), turned to -90 degrees
- moved ANT1 7.88 mm to (157.1, 76.6)
- moved TP1 7.56 mm to (157.3, 69.1)
- moved U9 7.56 mm to (164.8, 73.5)
- moved C37 5.23 mm to (182.8, 98.2)
- moved C40 3.38 mm to (180.3, 97.3)
- moved R39 3.33 mm to (180.3, 99.2)
- moved D8 2.27 mm to (177.8, 98.2)
- moved J4 1.07 mm to (127.1, 98.8)
Connections:
- U9 pad 7: Net-(JP1-A) -> unconnected-(U9-RESERVED-Pad7)
Routing:
- net /CPU_SWDCLK: track 0.00 -> 69.9 mm
- net /CPU_SWDIO: track 0.00 -> 61.3 mm
- net /SWCLK: track 0.00 -> 53.6 mm, vias 0 -> 2
- net /SWDIO: track 0.00 -> 50.6 mm, vias 0 -> 2
- net /UART1_TX_RADIO: track 0.00 -> 49.1 mm, vias 0 -> 1
- net /UART1_RX_RADIO: track 0.00 -> 48.1 mm, vias 0 -> 1
- net HIL_RX: track 0.00 -> 11.8 mm
- net HIL_TX: track 0.00 -> 9.33 mm
- net /RX_GPS: track 56.5 -> 64.8 mm, vias 1 -> 2
- net Net-(JP1-A): track 7.56 -> 0.00 mm
- net /L_RED: track 24.3 -> 16.9 mm, vias 1 -> 0
- net /TX_GPS: track 51.6 -> 58.8 mm, vias 1 -> 2
- net PPS: track 35.4 -> 41.6 mm
- net GND: track 0.00 -> 3.70 mm, vias 61 -> 67
- net /L_GREEN: track 19.8 -> 23.3 mm, vias 1 -> 0
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Other:
- board text added: "SWD-CPU"
- board text added: "SWD-RAK"
- board text added: "UART-HIL"
- board text added: "UART-RAK"

Commit message: Cristo risorto
Changed lines of the file:
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@@
 	)
 	(segment
-		(start 147.2238 106.5)
-		(end 139.5238 98.8)
+		(start 141.117592 100.393792)
+		(end 146.825628 106.101828)
 		(width 0.2245)
 		(layer "F.Cu")
@@
 	)
 	(segment
-		(start 139.5238 98.8)
+		(start 137.269836 98.8)
 		(end 130.1 98.8)
 		(width 0.2245)
@@
 	)
 	(segment
-		(start 148.35 106.5)
-		(end 147.2238 106.5)
+		(start 147.7869 106.5)
+		(end 148.35 106.5)
 		(width 0.2245)
 		(layer "F.Cu")
+		(net 23)
+	)
+	(arc
+		(start 141.117592 100.393792)
+		(mid 139.352226 99.214213)
+		(end 137.269836 98.8)
+		(width 0.2245)
+		(layer "F.Cu")
+		(net 23)
+	)
+	(arc
+		(start 146.825628 106.101828)
+		(mid 147.266663 106.396518)
+		(end 147.7869 106.5)
+		(width 0.2245)
+		(layer "F.Cu")
