File: microsd.kicad_sch (KiCad schematic)
At the start: 8 parts, among them J7 503398-1892

Commit message: robe di sabato che mi sono dimenticato di pushare
Connections:
- net +3V3: now also J7.10 (DETECT_SWITCH); no longer R40.1
- net GND: now also R40.1
- net micros_sd_detect: no longer J7.10 (DETECT_SWITCH)
Other:
- moved on the sheet: R40
Changed lines of the file:
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@@
+	)
+	(junction
+		(at 142.24 66.04)
+		(diameter 0)
+		(color 0 0 0 0)
+	)
+	(junction
+		(at 144.78 88.9)
+		(diameter 0)
+		(color 0 0 0 0)
+	)
+	(junction
+		(at 129.54 58.42)
+		(diameter 0)
+		(color 0 0 0 0)
+	)
+	(junction
+		(at 57.15 63.5)
+		(diameter 0)
+		(color 0 0 0 0)
+	)
+	(junction
+		(at 74.93 50.8)
+		(diameter 0)
+		(color 0 0 0 0)
+	)
+	(junction
+		(at 144.78 71.12)
+		(diameter 0)
+		(color 0 0 0 0)
+	)
+	(junction
+		(at 129.54 60.96)
+		(diameter 0)
+		(color 0 0 0 0)
+	)
+	(junction
+		(at 129.54 55.88)
+		(diameter 0)
+		(color 0 0 0 0)
+	)
+	(junction
+		(at 69.85 48.26)
+		(diameter 0)
+		(color 0 0 0 0)
+	)
+	(junction
+		(at 57.15 69.85)
+		(diameter 0)
+		(color 0 0 0 0)
+	)
+	(junction
+		(at 52.07 63.5)
+		(diameter 0)
+		(color 0 0 0 0)
+	)
+	(junction
+		(at 39.37 48.26)
+		(diameter 0)
+		(color 0 0 0 0)
+	)
+	(junction
+		(at 39.37 45.72)
+		(diameter 0)
+		(color 0 0 0 0)
+	)
+	(junction
+		(at 149.86 63.5)
+		(diameter 0)
+		(color 0 0 0 0)
+	)
+	(junction
+		(at 77.47 45.72)
+		(diameter 0)
+		(color 0 0 0 0)
 	)
 	(junction
@@
 		(color 0 0 0 0)
 	)
-	(junction
-		(at 142.24 66.04)
-		(diameter 0)
-		(color 0 0 0 0)
-	)
-	(junction
-		(at 144.78 88.9)
-		(diameter 0)
-		(color 0 0 0 0)
-	)
-	(junction
-		(at 134.62 48.26)
-		(diameter 0)
-		(color 0 0 0 0)
-	)
-	(junction
-		(at 129.54 58.42)
-		(diameter 0)
-		(color 0 0 0 0)
-	)
-	(junction
-		(at 57.15 63.5)
-		(diameter 0)
-		(color 0 0 0 0)
-	)
-	(junction
-		(at 74.93 50.8)
-		(diameter 0)
-		(color 0 0 0 0)
-	)
-	(junction
-		(at 144.78 71.12)
-		(diameter 0)
-		(color 0 0 0 0)
-	)
-	(junction
-		(at 129.54 60.96)
-		(diameter 0)
-		(color 0 0 0 0)
-	)
-	(junction
-		(at 129.54 55.88)
-		(diameter 0)
-		(color 0 0 0 0)
-	)
-	(junction
-		(at 69.85 48.26)
-		(diameter 0)
-		(color 0 0 0 0)
-	)
-	(junction
-		(at 57.15 69.85)
-		(diameter 0)
-		(color 0 0 0 0)
-	)
-	(junction
-		(at 52.07 63.5)
-		(diameter 0)
-		(color 0 0 0 0)
-	)
-	(junction
-		(at 39.37 48.26)
-		(diameter 0)
-		(color 0 0 0 0)
-	)
-	(junction
-		(at 39.37 45.72)
-		(diameter 0)
-		(color 0 0 0 0)
-	)
-	(junction
-		(at 149.86 63.5)
-		(diameter 0)
-		(color 0 0 0 0)
-	)
-	(junction
-		(at 77.47 45.72)
-		(diameter 0)
-		(color 0 0 0 0)
-	)
 	(no_connect
 		(at 147.32 74.93)
@@
 	(wire
 		(pts
-			(xy 134.62 48.26) (xy 153.67 48.26)
-		)
-		(stroke
-			(width 0)
-			(type default)
-		)
-	)
-	(wire
-		(pts
-			(xy 127 50.8) (xy 134.62 50.8)
+			(xy 127 50.8) (xy 132.08 50.8)
 		)
 		(stroke
@@
 	(wire
 		(pts
-			(xy 153.67 50.8) (xy 157.48 50.8)
+			(xy 153.67 48.26) (xy 157.48 48.26)
 		)
 		(stroke
@@
 	(wire
 		(pts
-			(xy 127 48.26) (xy 134.62 48.26)
+			(xy 127 48.26) (xy 153.67 48.26)
 		)
 		(stroke
@@
 	(wire
 		(pts
-			(xy 134.62 50.8) (xy 134.62 48.26)
-		)
-		(stroke
-			(width 0)
-			(type default)
-		)
-	)
-	(wire
-		(pts
 			(xy 144.78 71.12) (xy 161.29 71.12)
 		)
@@
 		(pts
 			(xy 69.85 39.37) (xy 69.85 48.26)
-		)
-		(stroke
-			(width 0)
-			(type default)
-		)
-	)
-	(wire
-		(pts
-			(xy 153.67 48.26) (xy 153.67 50.8)
 		)
 		(stroke
@@
 	(hierarchical_label "micros_sd_detect"
 		(shape input)
-		(at 157.48 50.8 0)
+		(at 157.48 48.26 0)
 		(effects
 			(font
@@
 	)
 	(symbol
+		(lib_id "power:GND")
+		(at 153.67 40.64 180)
+		(unit 1)
+		(exclude_from_sim no)
+		(in_bom yes)
+		(on_board yes)
+		(dnp no)
+		(fields_autoplaced yes)
+		(property "Reference" "#PWR0139"
+			(at 153.67 34.29 0)
+			(effects
+				(font
+					(size 1.27 1.27)
+				)
+				(hide yes)
+			)
+		)
+		(property "Value" "GND"
+			(at 153.67 35.56 0)
+			(effects
+				(font
+					(size 1.27 1.27)
+				)
+			)
+		)
+		(property "Footprint" ""
+			(at 153.67 40.64 0)
+			(effects
+				(font
+					(size 1.27 1.27)
+				)
+				(hide yes)
+			)
+		)
+		(property "Datasheet" ""
+			(at 153.67 40.64 0)
+			(effects
+				(font
+					(size 1.27 1.27)
+				)
+				(hide yes)
+			)
+		)
+		(property "Description" "Power symbol creates a global label with name \"GND\" , ground"
+			(at 153.67 40.64 0)
+			(effects
+				(font
+					(size 1.27 1.27)
+				)
+				(hide yes)
+			)
+		)
+		(pin "1"
+		)
+		(instances
+			(project "TABv1"
+				(path "/105f6e80-8e20-4d56-8eb3-6fa826818670/5f928ec3-de2c-45ad-87ae-24994ae19594"
+					(reference "#PWR0139")
+					(unit 1)
+				)
+			)
+		)
+	)
+	(symbol
 		(lib_id "microSD_503398-1892:503398-1892")
 		(at 83.82 45.72 0)
@@
 	(symbol
 		(lib_id "Device:R")
-		(at 157.48 48.26 270)
+		(at 153.67 44.45 0)
 		(unit 1)
 		(exclude_from_sim no)
@@
 		(dnp no)
 		(property "Reference" "R40"
-			(at 157.48 46.228 90)
+			(at 151.638 44.45 90)
 			(effects
 				(font
@@
 		)
 		(property "Value" "10k"
-			(at 157.48 48.26 90)
+			(at 153.67 44.45 90)
 			(effects
 				(font
@@
 		)
 		(property "Footprint" "Resistor_SMD:R_0603_1608Metric_Pad0.98x0.95mm_HandSolder"
-			(at 157.48 46.482 90)
+			(at 151.892 44.45 90)
 			(effects
 				(font
@@
 		)
 		(property "Datasheet" "~"
-			(at 157.48 48.26 0)
+			(at 153.67 44.45 0)
 			(effects
 				(font
@@
 		)
 		(property "Description" "Resistor"
-			(at 157.48 48.26 0)
+			(at 153.67 44.45 0)
 			(effects
 				(font
@@
 	(symbol
 		(lib_id "power:+3.3V")
-		(at 161.29 48.26 270)
+		(at 132.08 50.8 270)
 		(unit 1)
 		(exclude_from_sim no)
@@
 		(fields_autoplaced yes)
 		(property "Reference" "#PWR069"
-			(at 157.48 48.26 0)
+			(at 128.27 50.8 0)
 			(effects
 				(font
@@
 		)
 		(property "Value" "+3V3"
-			(at 165.1 48.2599 90)
+			(at 135.89 50.7999 90)
 			(effects
 				(font
@@
 		)
 		(property "Footprint" ""
-			(at 161.29 48.26 0)
+			(at 132.08 50.8 0)
 			(effects
 				(font
@@
 		)
 		(property "Datasheet" ""
-			(at 161.29 48.26 0)
+			(at 132.08 50.8 0)
 			(effects
 				(font
@@
 		)
 		(property "Description" "Power symbol creates a global label with name \"+3V3\""
-			(at 161.29 48.26 0)
+			(at 132.08 50.8 0)
 			(effects
 				(font
@@
 		)
 		(instances
-			(project "cockatiel"
+			(project "TABv1"
 				(path "/105f6e80-8e20-4d56-8eb3-6fa826818670/5f928ec3-de2c-45ad-87ae-24994ae19594"
 					(reference "#PWR069")

Commit message: Tentativo di Sbroglio
Connections:
- net +3V3: now also RN6.7 (R2.2), RN8.1 (R1.1), RN8.2 (R2.1), RN8.3 (R3.1), RN8.4 (R4.1); no longer RN8.5 (R4.2), RN8.6 (R3.2), RN8.8 (R1.2)
- net CLK: now also RN7.4 (R4.1); no longer RN9.7 (R2.2)
- net CMD: now also RN9.1 (R1.1); no longer RN7.6 (R3.2)
- net DAT0: now also RN7.3 (R3.1); no longer RN9.5 (R4.2)
- net DAT1: now also RN7.2 (R2.1); no longer RN9.8 (R1.2)
- net DAT2: now also RN9.3 (R3.1); no longer RN7.5 (R4.2)
- net DAT3: now also RN9.2 (R2.1); no longer RN7.8 (R1.2)
- net _DAT1: now also RN7.7 (R2.2), RN8.5 (R4.2); no longer RN8.1 (R1.1), RN9.1 (R1.1)
- net _DAT2: now also RN9.6 (R3.2); no longer RN7.4 (R4.1)
- net _DAT3: now also RN9.7 (R2.2); no longer RN7.1 (R1.1)
- net _CLK: now reaches RN8.7 (R2.2)
- net _CLK: now also J7.5 (CLK), RN7.5 (R4.2)
- net _CMD: now reaches RN6.2 (R2.1)
- net _CMD: now also J7.3 (CMD), RN9.8 (R1.2)
- new net _DAT0: J7.7 (DAT0), RN7.6 (R3.2), RN8.6 (R3.2)
- now unconnected: RN6.1 (R1.1), RN9.4 (R4.1)
- no-connect marks 8 -> 6
Other:
- moved on the sheet: C31, C32, J7, R40, RN6, RN7, RN8, RN9
